File: hardware/hotend_board/hotend_board.kicad_sch (KiCad schematic)
At the start: 0 parts

Commit message: update,
Parts:
- added J?: Print Cooling Fans, symbol Connector:Screw_Terminal_01x02
- added J?: Hotend Fan, symbol Connector:Screw_Terminal_01x02
- added J?: Z_Probe, symbol Connector:Screw_Terminal_01x03
- added J?: Hotend Heater, symbol Connector:Screw_Terminal_01x02
- added J?: Hotend Temp, symbol Connector:Screw_Terminal_01x02
- added U?: RJ45_NETWORK_SOCKET_1CH_LED, symbol my_connector_lib:RJ45_NETWORK_SOCKET_1CH_LED
Connections:
- new net +12V: J?.3 (Pin_3), U?.1.1
- new net COOLING_FANS_P: J?.2 (Pin_2), U?.1.4
- new net GND: J?.1 (Pin_1), J?.1 (Pin_1), J?.1 (Pin_1), J?.2 (Pin_2), U?.1.2
- new net HOTEND_FAN_P: J?.2 (Pin_2), U?.1.6
- new net HOTEND_HEATER_P: J?.2 (Pin_2), U?.1.5
- new net HOTEND_TEMP_N: J?.2 (Pin_2), U?.1.8
- new net HOTEND_TEMP_P: J?.1 (Pin_1), U?.1.7
- new net Z_PROBE: J?.1 (Pin_1), U?.1.3

Commit message: update,
Parts:
- added H1, H2, H3, H4: MountingHole, footprint-lib:MountingHole_3.1mm_M3,rpi_like, symbol Mechanical:MountingHole
- J1: renamed from J?; footprint (none) -> footprint-lib:PhoenixContact_MCV_1,5_3-G-5.08_1x03_P5.08mm_Vertical
- J2, J3, J4, J5: renamed from J?; footprint (none) -> footprint-lib:PhoenixContact_MCV_1,5_2-G-3.81_1x02_P3.81mm_Vertical
- U1: renamed from U?; footprint (none) -> my_connector_lib:RJ45_NETWORK_SOCKET_1CH_1_VERTICAL
